File: keyboard/keyboard.kicad_pcb (KiCad board)
At the start: 2 copper layers, 217.5 x 95.5 mm, 116 parts, among them SW1 SW_Push, SW10 SW_Push, SW11 SW_Push, SW12 SW_Push, SW13 SW_Push, SW14 SW_Push, SW15 SW_Push, SW16 SW_Push, SW17 SW_Push, SW18 SW_Push, SW19 SW_Push, SW2 SW_Push, SW20 SW_Push, SW21 SW_Push, SW22 SW_Push, SW23 SW_Push, SW24 SW_Push, SW25 SW_Push, SW26 SW_Push, SW27 SW_Push, SW28 SW_Push, SW29 SW_Push, SW3 SW_Push, SW30 SW_Push, SW31 SW_Push, SW32 SW_Push, SW33 SW_Push, SW34 SW_Push, SW35 SW_Push, SW36 SW_Push, SW37 SW_Push, SW38 SW_Push, SW39 SW_Push, SW4 SW_Push, SW40 SW_Push, SW41 SW_Push, SW42 SW_Push, SW43 SW_Push, SW44 SW_Push, SW45 SW_Push, SW46 SW_Push, SW47 SW_Push, SW48 SW_Push, SW49 SW_Push, SW5 SW_Push, SW50 SW_Push, SW51 SW_Push, SW52 SW_Push, SW53 SW_Push, SW54 SW_Push, SW55 SW_Push, SW56 SW_Push, SW6 SW_Push, SW7 SW_Push, SW8 SW_Push, SW9 SW_Push

Commit message: Add 3dshapes, footprint library, symbol library, and display mixer board.
Parts:
- added J1: Conn_01x22, kirdos:JUSHOU_AFC07-S20FCC-00-FPC-SMD_0.5P, F.Cu at (196.8, 22.7)
- moved D24 5.61 mm to (240.3, 60.2), turned to 0 degrees
- moved D36 5.60 mm to (240.3, 77.2), turned to 0 degrees
- moved D48 5.59 mm to (240.3, 94.2), turned to 0 degrees
- moved D12 5.59 mm to (240.3, 43.1), turned to 0 degrees
Connections:
- D12 pad 1: Row0 -> GND
- SW12 pad 1: Col11 -> Special
Routing:
- net Col0: track 58.1 -> 233.3 mm
- net Col1: track 58.1 -> 216.4 mm
- net Col2: track 77.8 -> 218.2 mm
- net Col3: track 77.5 -> 200.5 mm
- net Row4: track 128.0 -> 242.9 mm, vias 0 -> 2
- net Col4: track 77.5 -> 182.8 mm
- net Col5: track 77.5 -> 165.4 mm
- net Row3: track 200.0 -> 286.4 mm, vias 0 -> 2
- net Col6: track 77.5 -> 150.1 mm
- net Col7: track 77.5 -> 132.4 mm
- net Row2: track 199.8 -> 254.7 mm, vias 0 -> 2
- net Special: track 0.00 -> 43.2 mm
- net Col11: track 58.1 -> 98.5 mm, vias 0 -> 1
- net Col8: track 77.5 -> 113.5 mm
- net Row1: track 199.8 -> 232.6 mm, vias 0 -> 2
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- added copper zone on B.Cu, net GND
- added copper zone on F.Cu, net GND
Other:
- board text added: "2mm"
- board text added: "42mm"
- board text added: "Diodes on right side are inside to let the PCB slide into a groove"
- board text removed: "Diodes on right side are slightly closer to keep away from board edge"
- board text removed: "TODO: GND zones"

Commit message: Move main connector on display mixer and consolidate keyboard to single sheet.
Other:
- board text added: "81mm"
- board text removed: "82mm"
Changed lines of the file:
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@@
 				(font
 					(size 1.27 1.27)
+					(thickness 0.15)
 				)
 			)
@@
 		)
 	)
-	(gr_text "82mm"
+	(gr_text "81mm"
 		(at 31.95 97.175 0)
 		(layer "Cmts.User")
@@
 	)
 	(segment
+		(start 240.76 42.505101)
+		(end 240.76 43.15)
+		(width 0.2)
+		(layer "F.Cu")
+		(net "Net-(D12-A)")
+	)
+	(segment
+		(start 231.825 38.45)
+		(end 236.704899 38.45)
+		(width 0.2)
+		(layer "F.Cu")
+		(net "Net-(D12-A)")
+	)
+	(segment
+		(start 236.704899 38.45)
+		(end 240.76 42.505101)
+		(width 0.2)
+		(layer "F.Cu")
+		(net "Net-(D12-A)")
+	)
+	(segment
 		(start 105.825 106.45)
 		(end 117.6275 106.45)
@@
 	)
 	(segment
-		(start 240.76 42.505101)
-		(end 240.76 43.15)
-		(width 0.2)
-		(layer "F.Cu")
-		(net "Net-(D12-A)")
-	)
-	(segment
-		(start 231.825 38.45)
-		(end 236.704899 38.45)
-		(width 0.2)
-		(layer "F.Cu")
-		(net "Net-(D12-A)")
-	)
-	(segment
-		(start 236.704899 38.45)
-		(end 240.76 42.505101)
-		(width 0.2)
-		(layer "F.Cu")
-		(net "Net-(D12-A)")
-	)
-	(segment
